Commit message: added a left wheel

File: urdf/robot.urdf (robot description, URDF)
Before this commit: robot sphere_pusher, 1 links, 0 joints
Links:
- added link left_wheel; visual cylinder length=0.1 radius=0.05
Joints:
- added joint left_wheel_joint: type continuous, parent base_link, child left_wheel, origin xyz=-0.2 0.15 0 rpy=0 0 0, axis 0 1 0

Commit message: fixed the wheel position

File: urdf/robot.urdf (robot description, URDF)
Before this commit: robot sphere_pusher, 2 links, 1 joints
Links:
- link left_wheel: geometry visual cylinder length=0.05 radius=0.05
Joints:
- joint left_wheel_joint: limit (none) -> lower=0 upper=6.2832 effort=100 velocity=10; origin xyz=-0.2 0.15 0 rpy=0 0 0 -> xyz=-0.2 0.176 0 rpy=0 0 0; type continuous -> revolute

Commit message: Added a right wheel

File: urdf/robot.urdf (robot description, URDF)
Before this commit: robot sphere_pusher, 2 links, 1 joints
Links:
- added link right_wheel; visual cylinder length=0.05 radius=0.05
Joints:
- added joint right_wheel_joint: type revolute, parent base_link, child right_wheel, origin xyz=-0.2 -0.176 0 rpy=0 0 0, axis 0 1 0, limit lower=0 upper=6.2832 effort=100 velocity=10

Commit message: added a castor wheel

File: urdf/robot.urdf (robot description, URDF)
Before this commit: robot sphere_pusher, 3 links, 2 joints
Links:
- added link castor_wheel; visual sphere radius=0.03
Joints:
- added joint castor_wheel_joint: type fixed, parent base_link, child castor_wheel, origin xyz=0 0 -0.04 rpy=0 0 0

Commit message: Added inertial and collision tags for testing in gazebo

File: urdf/robot.urdf (robot description, URDF)
Before this commit: robot sphere_pusher, 4 links, 3 joints
Links:
- link base_link: mass None -> 5; geometry collision box size=0.5 0.3 0.1; visual box size=0.5 0.3 0.1
- link castor_wheel: mass None -> 0.2; geometry collision sphere radius=0.03; visual sphere radius=0.03
- link left_wheel: mass None -> 0.5; geometry collision cylinder length=0.05 radius=0.05; visual cylinder length=0.05 radius=0.05
- link right_wheel: mass None -> 0.5; geometry collision cylinder length=0.05 radius=0.05; visual cylinder length=0.05 radius=0.05
Joints:
- joint castor_wheel_joint: origin xyz=0 0 -0.04 rpy=0 0 0 -> xyz=0.17 0 -0.04 rpy=0 0 0
- joint left_wheel_joint: origin xyz=-0.2 0.176 0 rpy=0 0 0 -> xyz=-0.2 0.176 -0.04 rpy=0 0 0
- joint right_wheel_joint: origin xyz=-0.2 -0.176 0 rpy=0 0 0 -> xyz=-0.2 -0.176 -0.04 rpy=0 0 0

Commit message: added a dummy link to solve KDL issues

File: urdf/robot.urdf (robot description, URDF)
Before this commit: robot sphere_pusher, 4 links, 3 joints
Links:
- added link base_link_dummy, mass 0.01; collision sphere radius=0.01; visual sphere radius=0.01
- link base_link: mass 5 -> None
Joints:
- added joint base_to_dummy: type fixed, parent base_link, child base_link_dummy

Commit message: Fixed issue of robot moving about randomnly 1. increased inertia - no significant changes 2. reduced effort and velocity - corrected.

File: urdf/robot.urdf (robot description, URDF)
Before this commit: robot sphere_pusher, 5 links, 4 joints
Links:
- link base_link_dummy: mass 0.01 -> 1.0
Joints:
- joint left_wheel_joint: limit lower=0 upper=6.2832 effort=100 velocity=10 -> lower=0 upper=6.2832 effort=1 velocity=5
- joint right_wheel_joint: limit lower=0 upper=6.2832 effort=100 velocity=10 -> lower=0 upper=6.2832 effort=1 velocity=5
